File: PCB/connectors.kicad_sch (KiCad schematic)
At the start: 1 part, among them J1 Conn_01x02_Pin

Commit message: schematic
Parts:
- added J2, J3, J4: Conn_01x02_Pin, Connector_JST:JST_EH_B2B-EH-A_1x02_P2.50mm_Vertical, symbol Connector:Conn_01x02_Pin
Connections:
- new net OUTN_1: J3.2 (Pin_2)
- new net OUTN_2: J4.2 (Pin_2)
- new net OUTP_1: J3.1 (Pin_1)
- new net OUTP_2: J4.1 (Pin_1)
- new net RX_PICO: J2.2 (Pin_2)
- new net TX_PICO: J2.1 (Pin_1)
