File: PCB/mcu.kicad_sch (KiCad schematic)
At the start: 2 parts, among them U1 ESP32-S3-WROOM-1

Commit message: schematic
Parts:
- added J11: USB_C_Receptacle_USB2.0_16P, 0_LHRE_Footprints:USB-C_2.0_Receptacle, symbol Connector:USB_C_Receptacle_USB2.0_16P
- added R35, R8: 5.1k, Resistor_SMD:R_0603_1608Metric, symbol Device:R
Connections:
- net GND: now also J11.A1 (GND), J11.A12 (GND), J11.B1 (GND), J11.B12 (GND), R35.2, R8.2
- net USB_DN: now reaches U1.13 (USB_D-)
- net USB_DN: now also J11.A7 (D-), J11.B7 (D-)
- net USB_DP: now reaches U1.14 (USB_D+)
- net USB_DP: now also J11.A6 (D+), J11.B6 (D+)
- net I2S_DOUT: now reaches U1.17 (IO9)
- net I2S_BCLK: now reaches U1.18 (IO10)
- net I2S_LRCLK: now reaches U1.19 (IO11)
- net SD_MODE: now reaches U1.20 (IO12)
- new net: J11.A5 (CC1), R35.1
- new net: J11.B5 (CC2), R8.1
- new net USB_5V: J11.A4 (VBUS), J11.A9 (VBUS), J11.B4 (VBUS), J11.B9 (VBUS)
- no-connect marks 2 -> 31
Other:
- note added: "ESP32-S3-WROOM1"
- note added: "USB-C Connector"

Commit message: init layout
Parts:
- added R9: 100k, Resistor_SMD:R_0603_1608Metric, symbol Device:R
Connections:
- net +3V3: now also R9.1
- net SD_MODE: now also R9.2
Changed lines of the file:
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@@
+	)
+	(junction
+		(at 38.1 45.72)
+		(diameter 0)
+		(color 0 0 0 0)
 	)
 	(junction
@@
 	)
 	(junction
+		(at 22.86 83.82)
+		(diameter 0)
+		(color 0 0 0 0)
+	)
+	(junction
 		(at 146.05 59.69)
 		(diameter 0)
@@
 	(polyline
 		(pts
-			(xy 20.32 25.4) (xy 20.32 27.94)
+			(xy 13.97 25.4) (xy 13.97 27.94)
 		)
 		(stroke
@@
 	(wire
 		(pts
+			(xy 19.05 83.82) (xy 22.86 83.82)
+		)
+		(stroke
+			(width 0)
+			(type default)
+		)
+	)
+	(wire
+		(pts
 			(xy 146.05 62.23) (xy 146.05 59.69)
 		)
@@
 	(wire
 		(pts
-			(xy 38.1 48.26) (xy 38.1 43.18)
+			(xy 38.1 48.26) (xy 38.1 45.72)
 		)
 		(stroke
@@
 	(polyline
 		(pts
-			(xy 20.32 110.49) (xy 88.9 110.49)
+			(xy 13.97 110.49) (xy 88.9 110.49)
 		)
 		(stroke
@@
 	(wire
 		(pts
+			(xy 22.86 76.2) (xy 22.86 45.72)
+		)
+		(stroke
+			(width 0)
+			(type default)
+		)
+	)
+	(wire
+		(pts
 			(xy 133.35 74.93) (xy 134.62 74.93)
 		)
@@
 	(wire
 		(pts
+			(xy 38.1 45.72) (xy 38.1 43.18)
+		)
+		(stroke
+			(width 0)
+			(type default)
+		)
+	)
+	(wire
+		(pts
 			(xy 53.34 40.64) (xy 53.34 43.18)
 		)
@@
 	(polyline
 		(pts
-			(xy 88.9 25.4) (xy 20.32 25.4)
+			(xy 88.9 25.4) (xy 13.97 25.4)
+		)
+		(stroke
+			(width 0)
+			(type default)
+		)
+	)
+	(wire
+		(pts
+			(xy 22.86 45.72) (xy 38.1 45.72)
 		)
 		(stroke
@@
 	(polyline
 		(pts
-			(xy 20.32 26.67) (xy 20.32 110.49)
+			(xy 13.97 26.67) (xy 13.97 110.49)
 		)
 		(stroke
@@
 		(pts
 			(xy 134.62 72.39) (xy 138.43 72.39)
+		)
+		(stroke
+			(width 0)
+			(type default)
+		)
+	)
+	(wire
+		(pts
+			(xy 22.86 83.82) (xy 38.1 83.82)
 		)
 		(stroke
@@
 	(hierarchical_label "SD_MODE"
 		(shape output)
-		(at 38.1 83.82 180)
+		(at 19.05 83.82 270)
 		(effects
 			(font
@@
 		)
 	)
+	(symbol
+		(lib_id "Device:R")
+		(at 22.86 80.01 0)
+		(mirror y)
+		(unit 1)
+		(exclude_from_sim no)
+		(in_bom yes)
+		(on_board yes)
+		(dnp no)
+		(property "Reference" "R9"
+			(at 17.78 80.01 90)
+			(effects
+				(font
+					(size 1.27 1.27)
+				)
+			)
+		)
+		(property "Value" "100k"
+			(at 20.32 80.01 90)
+			(effects
+				(font
+					(size 1.27 1.27)
+				)
+			)
+		)
+		(property "Footprint" "Resistor_SMD:R_0603_1608Metric"
+			(at 24.638 80.01 90)
+			(effects
+				(font
+					(size 1.27 1.27)
+				)
+				(hide yes)
+			)
+		)
+		(property "Datasheet" ""
+			(at 22.86 80.01 0)
+			(effects
+				(font
+					(size 1.27 1.27)
+				)
+				(hide yes)
+			)
+		)
+		(property "Description" "Resistor"
+			(at 22.86 80.01 0)
+			(effects
+				(font
+					(size 1.27 1.27)
+				)
+				(hide yes)
+			)
+		)
+		(property "Mouser #" "603-RC0603FR-07100KL"
+			(at 22.86 80.01 0)
+			(effects
+				(font
+					(size 1.27 1.27)
+				)
+				(hide yes)
+			)
+		)
+		(property "Mouser Link" "https://www.mouser.com/ProductDetail/YAGEO/RC0603FR-07100KL?qs=e1ok2LiJcmaihem8Va5%2Fsw%3D%3D&srsltid=AfmBOooOdyEJhW55T0bTHCn9x1S_hWTbTVBciwDqFDvXTF-M6ZtkL9r2"
+			(at 22.86 80.01 0)
+			(effects
+				(font
+					(size 1.27 1.27)
+				)
+				(hide yes)
+			)
+		)
+		(property "JLCPCB #" "C14675"
+			(at 22.86 80.01 90)
+			(effects
+				(font
+					(size 1.27 1.27)
+				)
+				(hide yes)
+			)
+		)
+		(property "Mouser Part Number" "603-RC0603FR-07100KL"
+			(at 22.86 80.01 90)
+			(effects
+				(font
+					(size 1.27 1.27)
+				)
+				(hide yes)
+			)
+		)
+		(pin "2"
+		)
+		(pin "1"
+		)
+		(instances
+			(project "Hansoglasses"
+				(path "/565dd4cd-3458-4e26-8cb8-cc6b370af252/5d3d1737-fd18-4c19-965e-7a340bbed075"
+					(reference "R9")
+					(unit 1)
+				)
+			)
+		)
+	)
