File: PCB/power.kicad_sch (KiCad schematic)
At the start: 6 parts, among them U4 RT9013-33GB

Commit message: schematic
Parts:
- removed F9: 1A, Fuse:Fuse_0603_1608Metric_Pad1.05x0.95mm_HandSolder, symbol Device:Fuse
- added C5: 22u, Capacitor_SMD:C_0603_1608Metric, symbol Device:C
- added D20: D_Schottky, Diode_SMD:D_PowerDI-123, symbol Device:D_Schottky
- added F2: 1A, Fuse:Fuse_0603_1608Metric_Pad1.05x0.95mm_HandSolder, symbol Device:Fuse
- added SW1: SW_SPDT, Button_Switch_SMD:SW_SPDT_PCM12, symbol 0_LHRE_Symbols:SW_SPDT
Connections:
- net +5V: now also C5.1, F2.2
- net 5V_unfused: now also D20.1 (K), SW1.2 (B)
- net GND: now also C5.2
- new net: F2.1, SW1.1 (A)
- new net USB_+5V: D20.2 (A)
- no-connect marks 1 -> 2
Other:
- moved on the sheet: C1, C2, F1, TP3, U4

Commit message: init layout
Parts:
- removed TP3: GND, TestPoint:TestPoint_THTPad_1.5x1.5mm_Drill0.7mm, symbol Connector:TestPoint
Other:
- moved on the sheet: C5, D20, F2, SW1
