File: YerraGlasses/connectors.kicad_sch (KiCad schematic)
At the start: 5 parts, among them J1 Conn_01x02_Pin, J2 Conn_01x02_Pin, J3 Conn_01x02_Pin, J4 Conn_01x02_Pin, J5 Conn_01x02_Pin

Commit message: cad completion prototype
Connections:
- net 5V_unfused renamed 9V_unfused
Changed lines of the file:
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@@
 		)
 	)
-	(hierarchical_label "5V_unfused"
+	(hierarchical_label "9V_unfused"
 		(shape output)
 		(at 30.48 24.13 0)

Commit message: cad, pcb updaates
Parts:
- J1, J2, J3, J4, J5: footprint Connector_JST:JST_EH_B2B-EH-A_1x02_P2.50mm_Vertical -> Connector_JST:JST_PH_B2B-PH-K_1x02_P2.00mm_Vertical; JLCPCB # C160262 -> C131337; Mouser # 306-B2B-EH-A-GUP -> 306-B2BPHKSLFSNPP; Mouser Link https://www.mouser.com/ProductDetail/JST-Commercial/B2B-EH-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 -> https://www.mouser.com/ProductDetail/JST-Commercial/B2B-PH-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; Mouser Part Number 306-B2B-EH-A-GUP -> 306-B2BPHKSLFSNPP
