File: YerraGlasses/YerraGlasses.kicad_pcb (KiCad board)
At the start: 4 copper layers, 68 x 21.5 mm, 28 parts, among them J1 Conn_01x02_Pin, J11 USB_C_Receptacle_USB2.0_16P, J2 Conn_01x02_Pin, J3 Conn_01x02_Pin, J4 Conn_01x02_Pin, J5 Conn_01x02_Pin, SW1 SW_SPDT, U1 ESP32-S3-WROOM-1, U2 MAX98357A, U3 MAX98357A, U4 RT9013-33GB

Commit message: cad completion prototype
Parts:
- removed the REF** at (166.0, 43.0)
- removed the REF** at (166.0, 60.5)
- added ?: , , F.Cu at (159.8, 60.5)
- added REF**: MountingHole_2.2mm_M2_custom, MountingHole:MountingHole_2.2mm_M2_custom, F.Cu at (159.8, 43.0)
- added U6: R-78E5.0-1.0, Converter_DCDC:Converter_DCDC_RECOM_R-78E-0.5_THT, F.Cu at (164.5, 54.9)
Connections:
- D20 pad 1: /Connectors/5V_unfused -> /Power/5V_unfused
- F2 pad 1: Net-(SW1-A) -> /Power/5V_unfused
- J1 pad 1: /Connectors/5V_unfused -> /Connectors/9V_unfused
- SW1 pad 2: /Connectors/5V_unfused -> /Connectors/9V_unfused
Routing:
- net /Power/5V_unfused: track 0.00 -> 29.4 mm, vias 0 -> 1
- net Net-(SW1-A): track 3.85 -> 25.5 mm, vias 1 -> 0
- net /Connectors/5V_unfused: track 14.5 -> 0.00 mm, vias 1 -> 0
- net /Connectors/9V_unfused: track 0.00 -> 12.1 mm, vias 0 -> 1
- net GND: track 107.4 -> 110.6 mm, vias 27 -> 28
Other:
- board size 68 x 21.5 mm -> 74.5 x 21.5 mm

Commit message: updated cad, code start
Parts:
- removed ?: , 
- removed REF**: MountingHole_2.2mm_M2_custom, MountingHole:MountingHole_2.2mm_M2_custom
- added C15: 4.7u, Capacitor_SMD:C_1206_3216Metric_Pad1.33x1.80mm_HandSolder, B.Cu at (222.5, 49.5)
- added C4: 10u, Capacitor_SMD:C_0805_2012Metric, B.Cu at (186.8, 42.8)
Routing:
- net GND: track 110.6 -> 128.6 mm, vias 28 -> 35
- net +3V3: track 30.3 -> 32.7 mm

Commit message: updated pcb cad
Parts:
- added REF**: MountingHole_2.2mm_M2_custom, MountingHole:MountingHole_2.2mm_M2_custom, F.Cu at (159.8, 60.2)
- added REF**: MountingHole_2.2mm_M2_custom, MountingHole:MountingHole_2.2mm_M2_custom, F.Cu at (159.8, 43.2)
Changed lines of the file:
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@@
 		)
 	)
+	(footprint "MountingHole:MountingHole_2.2mm_M2_custom"
+		(layer "F.Cu")
+		(at 159.8 60.2)
+		(descr "Mounting Hole 2.2mm, M2, no annular, generated by kicad-footprint-generator mountinghole.py")
+		(tags "mountinghole M2")
+		(property "Reference" "REF**"
+			(at 0 -3.15 0)
+			(layer "F.SilkS")
+			(hide yes)
+			(effects
+				(font
+					(size 1 1)
+					(thickness 0.15)
+				)
+			)
+		)
+		(property "Value" "MountingHole_2.2mm_M2_custom"
+			(at 0 3.15 0)
+			(layer "F.Fab")
+			(hide yes)
+			(effects
+				(font
+					(size 1 1)
+					(thickness 0.15)
+				)
+			)
+		)
+		(property "Datasheet" ""
+			(at 0 0 0)
+			(layer "F.Fab")
+			(hide yes)
+			(effects
+				(font
+					(size 1.27 1.27)
+					(thickness 0.15)
+				)
+			)
+		)
+		(property "Description" ""
+			(at 0 0 0)
+			(layer "F.Fab")
+			(hide yes)
+			(effects
+				(font
+					(size 1.27 1.27)
+					(thickness 0.15)
+				)
+			)
+		)
+		(attr exclude_from_pos_files exclude_from_bom)
+		(fp_circle
+			(center 0 0)
+			(end 1.5 0)
+			(stroke
+				(width 0.15)
+				(type solid)
+			)
+			(fill no)
+			(layer "Cmts.User")
+		)
+		(pad "" np_thru_hole circle
+			(at 0 0)
+			(size 2.2 2.2)
+			(drill 2.2)
+			(layers "*.Cu" "*.Mask")
+		)
+		(embedded_fonts no)
+	)
 	(footprint "Connector_JST:JST_EH_B2B-EH-A_1x02_P2.50mm_Vertical"
 		(layer "F.Cu")
@@
 		)
 	)
+	(footprint "MountingHole:MountingHole_2.2mm_M2_custom"
+		(layer "F.Cu")
+		(at 159.8 43.2)
+		(descr "Mounting Hole 2.2mm, M2, no annular, generated by kicad-footprint-generator mountinghole.py")
+		(tags "mountinghole M2")
+		(property "Reference" "REF**"
+			(at 0 -3.15 0)
+			(layer "F.SilkS")
+			(hide yes)
+			(effects
+				(font
+					(size 1 1)
+					(thickness 0.15)
+				)
+			)
+		)
+		(property "Value" "MountingHole_2.2mm_M2_custom"
+			(at 0 3.15 0)
+			(layer "F.Fab")
+			(hide yes)
+			(effects
+				(font
+					(size 1 1)
+					(thickness 0.15)
+				)
+			)
+		)
+		(property "Datasheet" ""
+			(at 0 0 0)
+			(layer "F.Fab")
+			(hide yes)
+			(effects
+				(font
+					(size 1.27 1.27)
+					(thickness 0.15)
+				)
+			)
+		)
+		(property "Description" ""
+			(at 0 0 0)
+			(layer "F.Fab")
+			(hide yes)
+			(effects
+				(font
+					(size 1.27 1.27)
+					(thickness 0.15)
+				)
+			)
+		)
+		(attr exclude_from_pos_files exclude_from_bom)
+		(fp_circle
+			(center 0 0)
+			(end 1.5 0)
+			(stroke
+				(width 0.15)
+				(type solid)
+			)
+			(fill no)
+			(layer "Cmts.User")
+		)
+		(pad "" np_thru_hole circle
+			(at 0 0)
+			(size 2.2 2.2)
+			(drill 2.2)
+			(layers "*.Cu" "*.Mask")
+		)
+		(embedded_fonts no)
+	)
 	(footprint "Fuse:Fuse_0603_1608Metric_Pad1.05x0.95mm_HandSolder"

Commit message: cad, pcb updaates
Parts:
- removed REF** (x2): MountingHole_2.2mm_M2_custom, MountingHole:MountingHole_2.2mm_M2_custom
- added C9: 22u, Capacitor_SMD:C_0603_1608Metric_Pad1.08x0.95mm_HandSolder, B.Cu at (222.0, 48.6)
- added D32: Green, Diode_SMD:D_0603_1608Metric_Pad1.05x0.95mm_HandSolder, F.Cu at (168.8, 42.8)
- added D33: Green, Diode_SMD:D_0603_1608Metric_Pad1.05x0.95mm_HandSolder, F.Cu at (183.0, 49.0)
- added D5: SP3205-01ETG, 0_LHRE_Footprints:SP320501ETG, B.Cu at (160.0, 50.8)
- added D6: UDD32C05L01, Diode_SMD:D_SOD-323, B.Cu at (181.2, 56.2)
- added H1: MountingHole, MountingHole:MountingHole_2.2mm_M2_custom, F.Cu at (159.8, 43.2)
- added H2: MountingHole, MountingHole:MountingHole_2.2mm_M2_custom, F.Cu at (159.8, 60.2)
- added R1: 10k, Resistor_SMD:R_0603_1608Metric_Pad0.98x0.95mm_HandSolder, B.Cu at (221.6, 56.6)
- added R45: 10k, Resistor_SMD:R_0603_1608Metric_Pad0.98x0.95mm_HandSolder, B.Cu at (183.2, 49.0)
- added R46: 5.1k, Resistor_SMD:R_0603_1608Metric_Pad0.98x0.95mm_HandSolder, B.Cu at (163.3, 42.8)
- added R48: 5.1k, Resistor_SMD:R_0603_1608Metric_Pad0.98x0.95mm_HandSolder, B.Cu at (179.7, 49.0)
- added TP1: bootloader, TestPoint:TestPoint_Pad_1.0x1.0mm, F.Cu at (165.6, 59.8)
- added TP2: gndBootloader, TestPoint:TestPoint_Pad_1.0x1.0mm, F.Cu at (163.4, 59.8)
- C1, C2: footprint Capacitor_SMD:C_1206_3216Metric -> Capacitor_SMD:C_1206_3216Metric_Pad1.33x1.80mm_HandSolder
- C4, C8: footprint Capacitor_SMD:C_0805_2012Metric -> Capacitor_SMD:C_0805_2012Metric_Pad1.18x1.45mm_HandSolder
- C5: footprint Capacitor_SMD:C_0603_1608Metric -> Capacitor_SMD:C_0603_1608Metric_Pad1.08x0.95mm_HandSolder
- J1, J2, J3, J4, J5: footprint Connector_JST:JST_EH_B2B-EH-A_1x02_P2.50mm_Vertical -> Connector_JST:JST_PH_B2B-PH-K_1x02_P2.00mm_Vertical
- R35, R8, R9: footprint Resistor_SMD:R_0603_1608Metric -> Resistor_SMD:R_0603_1608Metric_Pad0.98x0.95mm_HandSolder
- moved C4 5.65 mm to (192.4, 42.6), turned to 180 degrees
- moved G*** 2.13 mm to (228.1, 53.0)
- moved C15 1.50 mm to (224.0, 49.4)
- moved J2 0.30 mm to (169.2, 49.2)
- moved J4 0.30 mm to (169.2, 58.5)
Connections:
- U1 pad 27: unconnected-(U1-IO0-Pad27) -> Net-(U1-IO0)
Routing:
- net Net-(U1-IO0): track 0.00 -> 58.0 mm, vias 0 -> 1
- net GND: track 128.6 -> 157.8 mm
- net +3V3: track 32.7 -> 51.9 mm, vias 5 -> 9
- net Net-(D33-A): track 0.00 -> 4.70 mm, vias 0 -> 1
- net +5V: track 20.7 -> 25.0 mm
- net Net-(D32-A): track 0.00 -> 3.83 mm, vias 0 -> 1
- net /MCU/USB_DP: track 18.4 -> 21.2 mm
- net Net-(R45-Pad1): track 0.00 -> 1.69 mm
- net /Connectors/OUTN_1: track 19.0 -> 17.8 mm
- net /Connectors/OUTN_2: track 35.4 -> 36.4 mm
- net /Connectors/OUTP_2: track 43.2 -> 44.1 mm
- net /Connectors/RX_PICO: track 46.9 -> 47.6 mm

Commit message: updated pcb order, cad
Parts:
- added C10: 100n, Capacitor_SMD:C_0603_1608Metric_Pad1.08x0.95mm_HandSolder, B.Cu at (203.8, 56.0)
- added C11: 100n, Capacitor_SMD:C_0603_1608Metric_Pad1.08x0.95mm_HandSolder, B.Cu at (163.6, 47.8)
- added JP1: SolderJumper_2_Open, Jumper:SolderJumper-2_P1.3mm_Open_RoundedPad1.0x1.5mm, F.Cu at (191.8, 47.6)
- added R2: 10k, Resistor_SMD:R_0603_1608Metric_Pad0.98x0.95mm_HandSolder, B.Cu at (199.8, 58.9)
- added R22: 22, Resistor_SMD:R_0603_1608Metric_Pad0.98x0.95mm_HandSolder, F.Cu at (201.8, 50.6)
- moved C6 1.14 mm to (219.2, 46.4)
- moved R1 1.11 mm to (220.5, 56.6), turned to 180 degrees
Connections:
- R1 pad 1: Net-(U1-IO0) -> +3V3
- R1 pad 2: +3V3 -> Net-(U1-IO0)
- U1 pad 3: +3V3 -> Net-(U1-EN)
- U2 pad 16: /MCU/I2S_BCLK -> /Speaker/BCLK_res
- U2 pad 2: +3V3 -> /Speaker/GAIN_SLOT
- U3 pad 16: /MCU/I2S_BCLK -> /Speaker/BCLK_res
- U3 pad 2: +3V3 -> /Speaker/GAIN_SLOT
Routing:
- net Net-(U1-EN): track 0.00 -> 29.3 mm, vias 0 -> 1
- net /Speaker/BCLK_res: track 0.00 -> 11.9 mm, vias 0 -> 2
- net /MCU/I2S_BCLK: track 15.5 -> 4.17 mm, vias 2 -> 0
- net /Speaker/GAIN_SLOT: track 0.00 -> 10.0 mm, vias 0 -> 1
- net GND: track 157.8 -> 164.6 mm
- net +3V3: track 51.9 -> 49.4 mm
- net /Power/5V_unfused: track 29.4 -> 31.5 mm
- net Net-(U1-IO0): track 58.0 -> 56.9 mm
Other:
- board text added: "#chwgparadise"
- board text added: "Rishi Bala Anh-Vu Nguyen"
