File: YerraGlasses/mcu.kicad_sch (KiCad schematic)
At the start: 6 parts, among them J11 USB_C_Receptacle_USB2.0_16P, U1 ESP32-S3-WROOM-1

Commit message: updated cad, code start
Parts:
- added C15: 4.7u, Capacitor_SMD:C_1206_3216Metric_Pad1.33x1.80mm_HandSolder, symbol Device:C
Connections:
- net +3V3: now also C15.1
- net GND: now also C15.2
Other:
- moved on the sheet: R9
Changed lines of the file:
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@@
 	)
 	(junction
-		(at 22.86 83.82)
+		(at 53.34 38.1)
 		(diameter 0)
 		(color 0 0 0 0)
@@
 		)
 	)
+	(wire
+		(pts
+			(xy 25.4 68.58) (xy 25.4 83.82)
+		)
+		(stroke
+			(width 0)
+			(type default)
+		)
+	)
 	(polyline
 		(pts
@@
 	(wire
 		(pts
-			(xy 19.05 83.82) (xy 22.86 83.82)
+			(xy 53.34 38.1) (xy 53.34 40.64)
 		)
 		(stroke
@@
 	(wire
 		(pts
-			(xy 22.86 76.2) (xy 22.86 45.72)
+			(xy 25.4 60.96) (xy 25.4 45.72)
 		)
 		(stroke
@@
 	(wire
 		(pts
-			(xy 53.34 35.56) (xy 53.34 40.64)
+			(xy 53.34 35.56) (xy 53.34 38.1)
 		)
 		(stroke
@@
 	(wire
 		(pts
-			(xy 22.86 45.72) (xy 38.1 45.72)
+			(xy 25.4 45.72) (xy 38.1 45.72)
 		)
 		(stroke
@@
 		)
 	)
+	(wire
+		(pts
+			(xy 25.4 83.82) (xy 38.1 83.82)
+		)
+		(stroke
+			(width 0)
+			(type default)
+		)
+	)
 	(polyline
 		(pts
@@
 		(pts
 			(xy 134.62 72.39) (xy 138.43 72.39)
-		)
-		(stroke
-			(width 0)
-			(type default)
-		)
-	)
-	(wire
-		(pts
-			(xy 22.86 83.82) (xy 38.1 83.82)
 		)
 		(stroke
@@
 	(hierarchical_label "SD_MODE"
 		(shape output)
-		(at 19.05 83.82 270)
+		(at 25.4 83.82 180)
 		(effects
 			(font
@@
 	)
 	(symbol
+		(lib_id "Device:C")
+		(at 57.15 38.1 90)
+		(unit 1)
+		(exclude_from_sim no)
+		(in_bom yes)
+		(on_board yes)
+		(dnp no)
+		(property "Reference" "C15"
+			(at 58.42 33.782 0)
+			(effects
+				(font
+					(size 1.27 1.27)
+				)
+				(justify left)
+			)
+		)
+		(property "Value" "4.7u"
+			(at 56.388 34.544 0)
+			(effects
+				(font
+					(size 1.27 1.27)
+				)
+				(justify left)
+			)
+		)
+		(property "Footprint" "Capacitor_SMD:C_1206_3216Metric_Pad1.33x1.80mm_HandSolder"
+			(at 60.96 37.1348 0)
+			(effects
+				(font
+					(size 1.27 1.27)
+				)
+				(hide yes)
+			)
+		)
+		(property "Datasheet" "~"
+			(at 57.15 38.1 0)
+			(effects
+				(font
+					(size 1.27 1.27)
+				)
+				(hide yes)
+			)
+		)
+		(property "Description" "Unpolarized capacitor"
+			(at 57.15 38.1 0)
+			(effects
+				(font
+					(size 1.27 1.27)
+				)
+				(hide yes)
+			)
+		)
+		(property "Mouser #" "187-CL31A475KBHNNNE"
+			(at 57.15 38.1 0)
+			(effects
+				(font
+					(size 1.27 1.27)
+				)
+				(hide yes)
+			)
+		)
+		(property "Mouser Link" "https://www.mouser.com/ProductDetail/Samsung-Electro-Mechanics/CL31A475KBHNNNE?qs=X6jEic%2FHinDAtDUeTge3nw%3D%3D"
+			(at 57.15 38.1 0)
+			(effects
+				(font
+					(size 1.27 1.27)
+				)
+				(hide yes)
+			)
+		)
+		(property "JLCPCB #" "C513768"
+			(at 57.15 38.1 0)
+			(effects
+				(font
+					(size 1.27 1.27)
+				)
+				(hide yes)
+			)
+		)
+		(pin "2"
+		)
+		(pin "1"
+		)
+		(instances
+			(project "YerraGlasses"
+				(path "/565dd4cd-3458-4e26-8cb8-cc6b370af252/5d3d1737-fd18-4c19-965e-7a340bbed075"
+					(reference "C15")
+					(unit 1)
+				)
+			)
+		)
+	)
+	(symbol
 		(lib_id "Device:R")
-		(at 22.86 80.01 0)
+		(at 25.4 64.77 0)
 		(mirror y)
 		(unit 1)
@@
 		(dnp no)
 		(property "Reference" "R9"
-			(at 17.78 80.01 90)
+			(at 20.32 64.77 90)
 			(effects
 				(font
@@
 		)
 		(property "Value" "100k"
-			(at 20.32 80.01 90)
+			(at 22.86 64.77 90)
 			(effects
 				(font
@@
 		)
 		(property "Footprint" "Resistor_SMD:R_0603_1608Metric"
-			(at 24.638 80.01 90)
+			(at 27.178 64.77 90)
 			(effects
 				(font
@@
 		)
 		(property "Datasheet" ""
-			(at 22.86 80.01 0)
+			(at 25.4 64.77 0)
 			(effects
 				(font
@@
 		)
 		(property "Description" "Resistor"
-			(at 22.86 80.01 0)
+			(at 25.4 64.77 0)
 			(effects
 				(font
@@
 		)
 		(property "Mouser #" "603-RC0603FR-07100KL"
-			(at 22.86 80.01 0)
+			(at 25.4 64.77 0)
 			(effects
 				(font
@@
 		)
 		(property "Mouser Link" "https://www.mouser.com/ProductDetail/YAGEO/RC0603FR-07100KL?qs=e1ok2LiJcmaihem8Va5%2Fsw%3D%3D&srsltid=AfmBOooOdyEJhW55T0bTHCn9x1S_hWTbTVBciwDqFDvXTF-M6ZtkL9r2"
-			(at 22.86 80.01 0)
+			(at 25.4 64.77 0)
 			(effects
 				(font
@@
 		)
 		(property "JLCPCB #" "C14675"
-			(at 22.86 80.01 90)
+			(at 25.4 64.77 90)
 			(effects
 				(font
@@
 		)
 		(property "Mouser Part Number" "603-RC0603FR-07100KL"
-			(at 22.86 80.01 90)
+			(at 25.4 64.77 90)
 			(effects
 				(font
@@
 					(unit 1)
 				)
+			)
+		)
+	)
+	(symbol
+		(lib_id "power:GND")
+		(at 60.96 38.1 90)
+		(unit 1)
+		(exclude_from_sim no)
+		(in_bom yes)
+		(on_board yes)
+		(dnp no)
+		(fields_autoplaced yes)
+		(property "Reference" "#PWR016"
+			(at 67.31 38.1 0)
+			(effects
+				(font
+					(size 1.27 1.27)
+				)
+				(hide yes)
+			)
+		)
+		(property "Value" "GND"
+			(at 64.77 38.0999 90)
+			(effects
+				(font
+					(size 1.27 1.27)
+				)
+				(justify right)
+			)
+		)
+		(property "Footprint" ""
+			(at 60.96 38.1 0)
+			(effects
+				(font
+					(size 1.27 1.27)
+				)
+				(hide yes)
+			)
+		)
+		(property "Datasheet" ""
+			(at 60.96 38.1 0)
+			(effects
+				(font
+					(size 1.27 1.27)
+				)
+				(hide yes)
+			)
+		)
+		(property "Description" "Power symbol creates a global label with name \"GND\" , ground"
+			(at 60.96 38.1 0)
+			(effects
+				(font
+					(size 1.27 1.27)
+				)
+				(hide yes)
+			)
+		)
+		(pin "1"
+		)
+		(instances
+			(project "YerraGlasses"
+				(path "/565dd4cd-3458-4e26-8cb8-cc6b370af252/5d3d1737-fd18-4c19-965e-7a340bbed075"
+					(reference "#PWR016")
+					(unit 1)
+				)

Commit message: cad, pcb updaates
Parts:
- added C9: 22u, Capacitor_SMD:C_0603_1608Metric_Pad1.08x0.95mm_HandSolder, symbol Device:C
- added H1, H2: MountingHole, MountingHole:MountingHole_2.2mm_M2_custom, symbol Mechanical:MountingHole
- added R1: 10k, Resistor_SMD:R_0603_1608Metric_Pad0.98x0.95mm_HandSolder, symbol Device:R
- added TP1: bootloader, TestPoint:TestPoint_Pad_1.0x1.0mm, symbol Connector:TestPoint
- added TP2: gndBootloader, TestPoint:TestPoint_Pad_1.0x1.0mm, symbol Connector:TestPoint
- R35, R8, R9: footprint Resistor_SMD:R_0603_1608Metric -> Resistor_SMD:R_0603_1608Metric_Pad0.98x0.95mm_HandSolder
Connections:
- net +3V3: now also C9.1, R1.2
- net GND: now also C9.2, TP2.1
- net at U1.27 (IO0): now also R1.1, TP1.1
- no-connect marks 31 -> 30
Other:
- moved on the sheet: C15

Commit message: updated pcb order, cad
Parts:
- added C10: 100n, Capacitor_SMD:C_0603_1608Metric_Pad1.08x0.95mm_HandSolder, symbol Device:C
- added R2: 10k, Resistor_SMD:R_0603_1608Metric_Pad0.98x0.95mm_HandSolder, symbol Device:R
- C15: Mouser Link https://www.mouser.com/ProductDetail/Samsung-Electro-Mechanics/CL31A475KBHNNNE?qs=X6jEic%2FHinDAtDUeTge3nw%3D%3D -> https://www.mouser.com/ProductDetail/Samsung-Electro-Mechanics/CL31A475KBHNNNE?qs=X6jEic%2FHinDAtDUeTge3nw%3D%3D&srsltid=AfmBOoqXGShmHEWF5TPyw7LucCVZ4UfmTiFjkyJX2UGL0MMP34FLKGAM; Mouser Part Number (none) -> 187-CL31A475KBHNNNE
- R1: Mouser Part Number (none) -> 71-CRCW0603-10K-E3
- TP1, TP2: now left out of the parts list
Connections:
- net +3V3: now also R1.1, R2.2; no longer R1.2, U1.3 (EN)
- net GND: now also C10.2
- net at TP1.1, U1.27 (IO0): now also R1.2; no longer R1.1
- new net: C10.1, R2.1, U1.3 (EN)
Other:
- moved on the sheet: R1, R9, TP1
