File: YerraGlasses/power.kicad_sch (KiCad schematic)
At the start: 8 parts, among them SW1 SW_SPDT, U4 RT9013-33GB

Commit message: cad completion prototype
Parts:
- added U6: R-78E5.0-1.0, Converter_DCDC:Converter_DCDC_RECOM_R-78E-0.5_THT, symbol Regulator_Switching:R-78E5.0-1.0
Connections:
- net 5V_unfused: now also F2.1, U6.3 (OUT); no longer SW1.2 (B)
- net GND: now also U6.2 (GND)
- net at SW1.1 (A): now also U6.1 (IN); no longer F2.1
- new net 9V_unfused: SW1.2 (B)
Other:
- note added: "5V safety"
- note added: "9V to 5V Switching Regulator"
- moved on the sheet: C1, C2, C5, D20, F1, F2, SW1, U4

Commit message: cad, pcb updaates
Parts:
- added D32, D33: Green, Diode_SMD:D_0603_1608Metric_Pad1.05x0.95mm_HandSolder, symbol Device:LED
- added D5: SP3205-01ETG, 0_LHRE_Footprints:SP320501ETG, symbol shuttle_parts:SP3205-01ETG
- added D6: UDD32C05L01, Diode_SMD:D_SOD-323, symbol shuttle_parts:PESD5V0X1BCSFYL
- added R45: 10k, Resistor_SMD:R_0603_1608Metric_Pad0.98x0.95mm_HandSolder, symbol Device:R
- added R46, R48: 5.1k, Resistor_SMD:R_0603_1608Metric_Pad0.98x0.95mm_HandSolder, symbol Device:R
- C1, C2: footprint Capacitor_SMD:C_1206_3216Metric -> Capacitor_SMD:C_1206_3216Metric_Pad1.33x1.80mm_HandSolder
- C5: footprint Capacitor_SMD:C_0603_1608Metric -> Capacitor_SMD:C_0603_1608Metric_Pad1.08x0.95mm_HandSolder
Connections:
- net +3V3: now also D5.1, R46.2
- net +5V: now also D6.2, R45.2
- net GND: now also D32.1 (K), D33.1 (K), D5.2, D6.1
- new net: D32.2 (A), R46.1
- new net: R45.1, R48.2
- new net: D33.2 (A), R48.1
Other:
- note added: "Power Indicators"

Commit message: updated pcb order, cad
Parts:
- added C11: 100n, Capacitor_SMD:C_0603_1608Metric_Pad1.08x0.95mm_HandSolder, symbol Device:C
- D32, D33: Mouser Part Number (none) -> 604-APT1608LZGCK
- D5: Mouser Part Number (none) -> 576-SP3205-01ETG
- D6: Mouser Part Number (none) -> 603-UDD32C05L01
- R45: Mouser Part Number (none) -> 71-CRCW0603-10K-E3
Connections:
- net 5V_unfused: now also C11.2
- net GND: now also C11.1
- net USB_+5V renamed USB_5V
